File: KiCAD/pathfinder.kicad_sch (KiCad schematic)
At the start: 3 parts, among them SW1 SW_Push, U1 MOUDLE-SEEEDUINO-XIAO

Commit message: treasure map
Parts:
- added D2, D3: LED, symbol Device:LED
- added SW2, SW3: SW_Push, symbol Switch:SW_Push
Other:
- moved on the sheet: SW1, U1

Commit message: schematic tutorial
Parts:
- removed D1, D2, D3: LED, symbol Device:LED
- removed U1: MOUDLE-SEEEDUINO-XIAO, symbol XIAO_RP2040:MOUDLE-SEEEDUINO-XIAO
- added D1, D2, D3: L08R5000Q1, L08R5000Q1:LEDRD254W57D500H1070, symbol L08R5000Q1:L08R5000Q1
- added R1, R2, R3: R, symbol Device:R
- added U1: XIAO-RP2040-DIP, Module:MOUDLE14P-XIAO-DIP-SMD, symbol Seeed_Studio_XIAO_Series:XIAO-RP2040-DIP
Connections:
- net button2: now reaches SW2.1
- net button2: now also U1.2 (GPIO27/ADC1/A1)
- net GND: now reaches SW2.2
- net GND: now also SW1.2, SW3.2, D1.C, D2.C, D3.C, U1.13 (GND)
- net button1: now reaches SW1.1
- net button1: now also U1.1 (GPIO26/ADC0/A0)
- net button3: now reaches SW3.1
- net button3: now also U1.3 (GPIO28/ADC2/A2)
- new net: D1.A, R1.1
- new net: D3.A, R3.1
- new net: D2.A, R2.1
- new net LED1: R1.2, U1.4 (GPIO29/ADC3/A3)
- new net LED2: R2.2, U1.5 (GPIO6/SDA)
- new net LED3: R3.2, U1.6 (GPIO7/SCL)

Commit message: pcb making + firmware
Parts:
- D1, D2, D3: footprint L08R5000Q1:LEDRD254W57D500H1070 -> footprints:LEDRD254W57D500H1070
- R1, R2, R3: footprint (none) -> Resistor_THT:R_Axial_DIN0204_L3.6mm_D1.6mm_P5.08mm_Horizontal
- SW1, SW2, SW3: footprint (none) -> Button_Switch_Keyboard:SW_Cherry_MX_1.00u_PCB
- U1: footprint Module:MOUDLE14P-XIAO-DIP-SMD -> footprints:XIAO-RP2040-DIP
Other:
- company: (none) -> Hack Club
- title: (none) -> Pathfinder
Changed lines of the file:
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@@
 	(generator_version "9.0")
 	(paper "A4")
+	(title_block
+		(title "Pathfinder")
+		(date "6/24/2025")
+		(rev "6/26/2025")
+		(company "Hack Club")
+	)
 	(wire
 		(pts
@@
 			)
 		)
-		(property "Footprint" ""
+		(property "Footprint" "Button_Switch_Keyboard:SW_Cherry_MX_1.00u_PCB"
 			(at 82.55 66.675 0)
 			(effects
@@
 			)
 		)
-		(property "Footprint" ""
+		(property "Footprint" "Resistor_THT:R_Axial_DIN0204_L3.6mm_D1.6mm_P5.08mm_Horizontal"
 			(at 89.662 90.805 90)
 			(effects
@@
 			)
 		)
-		(property "Footprint" ""
+		(property "Footprint" "Resistor_THT:R_Axial_DIN0204_L3.6mm_D1.6mm_P5.08mm_Horizontal"
 			(at 127.762 90.805 90)
 			(effects
@@
 			)
 		)
-		(property "Footprint" ""
+		(property "Footprint" "Resistor_THT:R_Axial_DIN0204_L3.6mm_D1.6mm_P5.08mm_Horizontal"
 			(at 109.347 90.805 90)
 			(effects
@@
 			)
 		)
-		(property "Footprint" "L08R5000Q1:LEDRD254W57D500H1070"
+		(property "Footprint" "footprints:LEDRD254W57D500H1070"
 			(at 137.16 86.995 0)
 			(effects
@@
 			)
 		)
-		(property "Footprint" "L08R5000Q1:LEDRD254W57D500H1070"
+		(property "Footprint" "footprints:LEDRD254W57D500H1070"
 			(at 99.06 86.995 0)
 			(effects
@@
 			)
 		)
-		(property "Footprint" "L08R5000Q1:LEDRD254W57D500H1070"
+		(property "Footprint" "footprints:LEDRD254W57D500H1070"
 			(at 118.745 86.995 0)
 			(effects
@@
 			)
 		)
-		(property "Footprint" ""
+		(property "Footprint" "Button_Switch_Keyboard:SW_Cherry_MX_1.00u_PCB"
 			(at 109.855 66.04 0)
 			(effects
@@
 			)
 		)
-		(property "Footprint" ""
+		(property "Footprint" "Button_Switch_Keyboard:SW_Cherry_MX_1.00u_PCB"
 			(at 136.525 66.675 0)
 			(effects
@@
 			)
 		)
-		(property "Footprint" "Module:MOUDLE14P-XIAO-DIP-SMD"
+		(property "Footprint" "footprints:XIAO-RP2040-DIP"
 			(at 112.268 136.398 0)
 			(effects
